Commit message: now working

File: install/mobile_robot/share/mobile_robot/model/robot.xacro (robot description, xacro)
@@ -5,189 +5,254 @@
 <!-- ####################### -->
 <robot name="differential_drive_robot" xmlns:xacro="http://www.ros.org/wiki/xacro">
-<!-- Body Dimensions -->
-<xacro:property name="body_link_x_dim" value="1"/>
-<xacro:property name="body_link_y_dim" value="0.6"/>
-<xacro:property name="body_link_z_dim" value="0.3"/>
-<!-- Wheel Dimensions -->
-<xacro:property name="wheel_link_radius" value="0.15"/>
-<xacro:property name="wheel_link_length" value="0.1"/>
-<xacro:property name="wheel_link_z_location" value="-0.1"/>
-<!-- Material Density -->
-<xacro:property name="body_density" value="2710.0"/>
-<xacro:property name="wheel_density" value="2710.0"/>
-<!-- PI constant -->
-<xacro:property name="pi_const" value="3.14159265"/>
-<!-- Robot body and wheel mass -->
-<xacro:property name="body_mass" value="${body_density*body_link_x_dim*body_link_y_dim*body_link_z_dim}"/>
-<xacro:property name="wheel_mass" value="${wheel_density*pi_const*wheel_link_length*wheel_link_radius*wheel_link_radius}"/>
-<!-- Moments of Inertia of the wheel -->
-<xacro:property name="Iz_wheel" value="${0.5*wheel_mass*wheel_link_radius*wheel_link_radius}"/>
-<xacro:property name="I_wheel" value="${(1.0/12.0)*wheel_mass*(3.0*wheel_link_radius*wheel_link_radius+wheel_link_length*wheel_link_length)}"/>
-<!-- This macro defines the inertial section of the wheel -->
-<xacro:macro name="inertia_wheel">
-<inertial>
-    <origin rpy="0 0 0" xyz="0 0 0"/>
-    <mass value="${wheel_mass}"/>
-    <inertia ixx="${I_wheel}" ixy="0.0" ixz="0.0" iyy="${I_wheel}" iyz="0" izz="${Iz_wheel}"/>
-</inertial>
-</xacro:macro>
-<!-- Over here we include the file that defines extra Gazebo option and robot control driver -->
-<xacro:include filename="$(find mobile_robot)/model/robot.gazebo"/>
-<!-- ####################### -->
-<!-- DEFINE LINKS AND JOINTS -->
-<!-- ####################### -->
-<!-- necessary dummy -->
-<link name="dummy">
+    <!-- Body Dimensions -->
+    <xacro:property name="body_link_x_dim" value="1" />
+    <xacro:property name="body_link_y_dim" value="0.6" />
+    <xacro:property name="body_link_z_dim" value="0.3" />
+    <!-- Wheel Dimensions -->
+    <xacro:property name="wheel_link_radius" value="0.15" />
+    <xacro:property name="wheel_link_length" value="0.1" />
+    <xacro:property name="wheel_link_z_location" value="-0.1" />
+    <!-- Material Density -->
+    <xacro:property name="body_density" value="2710.0" />
+    <xacro:property name="wheel_density" value="2710.0" />
+    <!-- PI constant -->
+    <xacro:property name="pi_const" value="3.14159265" />
+    <!-- Robot body and wheel mass -->
+    <xacro:property name="body_mass"
+        value="${body_density*body_link_x_dim*body_link_y_dim*body_link_z_dim}" />
+    <xacro:property name="wheel_mass"
+        value="${wheel_density*pi_const*wheel_link_length*wheel_link_radius*wheel_link_radius}" />
+    <!-- Moments of Inertia of the wheel -->
+    <xacro:property name="Iz_wheel" value="${0.5*wheel_mass*wheel_link_radius*wheel_link_radius}" />
+    <xacro:property name="I_wheel"
+        value="${(1.0/12.0)*wheel_mass*(3.0*wheel_link_radius*wheel_link_radius+wheel_link_length*wheel_link_length)}" />
+    <xacro:property name="camera_link" value="0.05" /> <!-- Size of square 'camera' box -->
+    <!-- This macro defines the inertial section of the wheel -->
+    <xacro:macro name="inertia_wheel">
+        <inertial>
+            <origin rpy="0 0 0" xyz="0 0 0" />
+            <mass value="${wheel_mass}" />
+            <inertia ixx="${I_wheel}" ixy="0.0" ixz="0.0" iyy="${I_wheel}" iyz="0" izz="${Iz_wheel}" />
+        </inertial>
+    </xacro:macro>
+    <!-- Over here we include the file that defines extra Gazebo option and robot control driver -->
+    <xacro:include filename="$(find mobile_robot)/model/robot.gazebo" />
+    <!-- ####################### -->
+    <!-- DEFINE LINKS AND JOINTS -->
+    <!-- ####################### -->
+    <!-- necessary dummy -->
+    <link name="dummy">
 </link>
-<joint name="dummy_joint" type="fixed">
-    <parent link="dummy"/>
-    <child link="body_link"/>
-</joint>
-<!-- ####################### -->
-<!-- Start: Body link of the robot-->
-<!-- ####################### -->
-<link name="body_link">
-    <visual>
-        <geometry>
-            <box size="${body_link_x_dim} ${body_link_y_dim} ${body_link_z_dim}"/>
-        </geometry>
-        <origin rpy="0 0 0" xyz="0 0 0"/>
-    </visual>
-    <collision>
-        <geometry>
-            <box size="${body_link_x_dim} ${body_link_y_dim} ${body_link_z_dim}"/>
-        </geometry>
-        <origin rpy="0 0 0" xyz="0 0 0"/>
-    </collision>
-    <inertial>
-        <origin rpy="0 0 0" xyz="0 0 0"/>
-        <mass value="${body_mass}"/>
-        <inertia
-            ixx="${(1/12)*body_mass*(body_link_y_dim*body_link_y_dim+body_link_z_dim*body_link_z_dim)}"
-            ixy="0"
-            ixz="0"
-            iyy="${(1/12)*body_mass*(body_link_x_dim*body_link_x_dim+body_link_z_dim*body_link_z_dim)}"
-            iyz="0"
-            izz="${(1/12)*body_mass*(body_link_y_dim*body_link_y_dim+body_link_x_dim*body_link_x_dim)}"/>
-    </inertial>
-</link>
-<!-- ####################### -->
-<!-- END: Body link of the robot-->
-<!-- ####################### -->
-<!-- ####################### -->
-<!-- Start: Back right wheel of the robot and the joint-->
-<!-- ####################### -->
-<joint name="wheel1_joint" type="continuous">
-    <parent link="body_link"/>
-    <child link="wheel1_link"/>
-    <origin xyz="${-body_link_x_dim/2 +1.2*wheel_link_radius} ${-body_link_y_dim/2-wheel_link_length/2} ${wheel_link_z_location}" rpy="0 0 0"/>
-    <axis xyz="0 1 0"/>
-    <limit effort="1000" velocity="1000"/>
-    <dynamics damping="1.0" friction="1.0"/>
-</joint>
-<link name="wheel1_link">
-    <visual>
-        <geometry>
-            <cylinder length = "${wheel_link_length}" radius="${wheel_link_radius}"/>
-        </geometry>
-    <origin rpy="${pi_const/2} 0 0" xyz="0 0 0"/>
-    </visual>
-    <collision>
-        <geometry>
-           <cylinder length = "${wheel_link_length}" radius="${wheel_link_radius}"/>
-        </geometry>
-    <origin rpy="${pi_const/2} 0 0" xyz="0 0 0"/>
-    </collision>
-    <xacro:inertia_wheel/>
- </link>
-<!-- ####################### -->
-<!-- END:Right back wheel and joint-->
-<!-- ####################### -->
-<!-- ####################### -->
-<!-- Start: Back left wheel of the robot and the joint-->
-<!-- ####################### -->
-<joint name="wheel2_joint" type="continuous">
-    <parent link="body_link"/>
-    <child link="wheel2_link"/>
-    <origin xyz="${-body_link_x_dim/2 +1.2*wheel_link_radius} ${body_link_y_dim/2+wheel_link_length/2} ${wheel_link_z_location}" rpy="0 0 0"/>
-    <axis xyz="0 1 0"/>
-    <limit effort="1000" velocity="1000"/>
-    <dynamics damping="1.0" friction="1.0"/>
-</joint>
-<link name="wheel2_link">
-    <visual>
-        <geometry>
-            <cylinder length="${wheel_link_length}" radius="${wheel_link_radius}"/>
-        </geometry>
-        <origin rpy="${pi_const/2} 0 0" xyz="0 0 0"/>
-    </visual>
-    <collision>
-        <geometry>
-           <cylinder length="${wheel_link_length}" radius="${wheel_link_radius}"/>
-        </geometry>
-        <origin rpy="${pi_const/2} 0 0" xyz="0 0 0"/>
-    </collision>
-    <xacro:inertia_wheel/>
-</link>
-<!-- ####################### -->
-<!-- END: Left back wheel and joint-->
-<!-- ####################### -->
-<!-- ####################### -->
-<!-- Start: Front right wheel of the robot and the joint-->
-<!-- ####################### -->
-<joint name="wheel3_joint" type="continuous">
-    <parent link="body_link"/>
-    <child link="wheel3_link"/>
-    <origin xyz="${body_link_x_dim/2 -1.2*wheel_link_radius} ${-body_link_y_dim/2-wheel_link_length/2} ${wheel_link_z_location}" rpy="0 0 0"/>
-    <axis xyz="0 1 0"/>
-    <limit effort="1000" velocity="1000"/>
-    <dynamics damping="1.0" friction="1.0"/>
-</joint>
-<link name="wheel3_link">
-    <visual>
-        <geometry>
-            <cylinder length="${wheel_link_length}" radius="${wheel_link_radius}"/>
-        </geometry>
-        <origin rpy="${pi_const/2} 0 0" xyz="0 0 0"/>
-    </visual>
-    <collision>
-        <geometry>
-           <cylinder length="${wheel_link_length}" radius="${wheel_link_radius}"/>
-        </geometry>
-        <origin rpy="${pi_const/2} 0 0" xyz="0 0 0"/>
-    </collision>
-    <xacro:inertia_wheel/>
-</link>
-<!-- ####################### -->
-<!-- END: Right front wheel and joint-->
-<!-- ####################### -->
-<!-- ####################### -->
-<!-- Start: Front left wheel of the robot and the joint-->
-<!-- ####################### -->
-<joint name="wheel4_joint" type="continuous">
-    <parent link="body_link"/>
-    <child link="wheel4_link"/>
-    <origin xyz="${body_link_x_dim/2 -1.2*wheel_link_radius} ${body_link_y_dim/2+wheel_link_length/2} ${wheel_link_z_location}" rpy="0 0 0"/>
-    <axis xyz="0 1 0"/>
-    <limit effort="1000" velocity="1000"/>
-    <dynamics damping="1.0" friction="1.0"/>
-</joint>
-<link name="wheel4_link">
-    <visual>
-        <geometry>
-            <cylinder length="${wheel_link_length}" radius="${wheel_link_radius}"/>
-        </geometry>
-        <origin rpy="${pi_const/2} 0 0" xyz="0 0 0"/>
-    </visual>
-    <collision>
-        <geometry>
-           <cylinder length="${wheel_link_length}" radius="${wheel_link_radius}"/>
-        </geometry>
-        <origin rpy="${pi_const/2} 0 0" xyz="0 0 0"/>
-    </collision>
-    <xacro:inertia_wheel/>
-</link>
-<!-- ####################### -->
-<!-- END: Left front wheel and joint-->
-<!-- ####################### -->
+    <joint name="dummy_joint" type="fixed">
+        <parent link="dummy" />
+        <child link="body_link" />
+    </joint>
+    <!-- ####################### -->
+    <!-- Start: Body link of the robot-->
+    <!-- ####################### -->
+    <link name="body_link">
+        <visual>
+            <geometry>
+                <box size="${body_link_x_dim} ${body_link_y_dim} ${body_link_z_dim}" />
+            </geometry>
+            <origin rpy="0 0 0" xyz="0 0 0" />
+        </visual>
+        <collision>
+            <geometry>
+                <box size="${body_link_x_dim} ${body_link_y_dim} ${body_link_z_dim}" />
+            </geometry>
+            <origin rpy="0 0 0" xyz="0 0 0" />
+        </collision>
+        <inertial>
+            <origin rpy="0 0 0" xyz="0 0 0" />
+            <mass value="${body_mass}" />
+            <inertia
+                ixx="${(1/12)*body_mass*(body_link_y_dim*body_link_y_dim+body_link_z_dim*body_link_z_dim)}"
+                ixy="0"
+                ixz="0"
+                iyy="${(1/12)*body_mass*(body_link_x_dim*body_link_x_dim+body_link_z_dim*body_link_z_dim)}"
+                iyz="0"
+                izz="${(1/12)*body_mass*(body_link_y_dim*body_link_y_dim+body_link_x_dim*body_link_x_dim)}" />
+        </inertial>
+    </link>
+    <!-- ####################### -->
+    <!-- END: Body link of the robot-->
+    <!-- ####################### -->
+    <!-- ####################### -->
+    <!-- Start: Back right wheel of the robot and the joint-->
+    <!-- ####################### -->
+    <joint name="wheel1_joint" type="continuous">
+        <parent link="body_link" />
+        <child link="wheel1_link" />
+        <origin
+            xyz="${-body_link_x_dim/2 +1.2*wheel_link_radius} ${-body_link_y_dim/2-wheel_link_length/2} ${wheel_link_z_location}"
+            rpy="0 0 0" />
+        <axis xyz="0 1 0" />
+        <limit effort="1000" velocity="1000" />
+        <dynamics damping="1.0" friction="1.0" />
+    </joint>
+    <link name="wheel1_link">
+        <visual>
+            <geometry>
+                <cylinder length="${wheel_link_length}" radius="${wheel_link_radius}" />
+            </geometry>
+            <origin rpy="${pi_const/2} 0 0" xyz="0 0 0" />
+        </visual>
+        <collision>
+            <geometry>
+                <cylinder length="${wheel_link_length}" radius="${wheel_link_radius}" />
+            </geometry>
+            <origin rpy="${pi_const/2} 0 0" xyz="0 0 0" />
+        </collision>
+        <xacro:inertia_wheel />
+    </link>
+    <!-- ####################### -->
+    <!-- END:Right back wheel and joint-->
+    <!-- ####################### -->
+    <!-- ####################### -->
+    <!-- Start: Back left wheel of the robot and the joint-->
+    <!-- ####################### -->
+    <joint name="wheel2_joint" type="continuous">
+        <parent link="body_link" />
+        <child link="wheel2_link" />
+        <origin
+            xyz="${-body_link_x_dim/2 +1.2*wheel_link_radius} ${body_link_y_dim/2+wheel_link_length/2} ${wheel_link_z_location}"
+            rpy="0 0 0" />
+        <axis xyz="0 1 0" />
+        <limit effort="1000" velocity="1000" />
+        <dynamics damping="1.0" friction="1.0" />
+    </joint>
+    <link name="wheel2_link">
+        <visual>
+            <geometry>
+                <cylinder length="${wheel_link_length}" radius="${wheel_link_radius}" />
+            </geometry>
+            <origin rpy="${pi_const/2} 0 0" xyz="0 0 0" />
+        </visual>
+        <collision>
+            <geometry>
+                <cylinder length="${wheel_link_length}" radius="${wheel_link_radius}" />
+            </geometry>
+            <origin rpy="${pi_const/2} 0 0" xyz="0 0 0" />
+        </collision>
+        <xacro:inertia_wheel />
+    </link>
+    <!-- ####################### -->
+    <!-- END: Left back wheel and joint-->
+    <!-- ####################### -->
+    <!-- ####################### -->
+    <!-- Start: Front right wheel of the robot and the joint-->
+    <!-- ####################### -->
+    <joint name="wheel3_joint" type="continuous">
+        <parent link="body_link" />
+        <child link="wheel3_link" />
+        <origin
+            xyz="${body_link_x_dim/2 -1.2*wheel_link_radius} ${-body_link_y_dim/2-wheel_link_length/2} ${wheel_link_z_location}"
+            rpy="0 0 0" />
+        <axis xyz="0 1 0" />
+        <limit effort="1000" velocity="1000" />
+        <dynamics damping="1.0" friction="1.0" />
+    </joint>
+    <link name="wheel3_link">
+        <visual>
+            <geometry>
+                <cylinder length="${wheel_link_length}" radius="${wheel_link_radius}" />
+            </geometry>
+            <origin rpy="${pi_const/2} 0 0" xyz="0 0 0" />
+        </visual>
+        <collision>
+            <geometry>
+                <cylinder length="${wheel_link_length}" radius="${wheel_link_radius}" />
+            </geometry>
+            <origin rpy="${pi_const/2} 0 0" xyz="0 0 0" />
+        </collision>
+        <xacro:inertia_wheel />
+    </link>
+    <!-- ####################### -->
+    <!-- END: Right front wheel and joint-->
+    <!-- ####################### -->
+    <!-- ####################### -->
+    <!-- Start: Front left wheel of the robot and the joint-->
+    <!-- ####################### -->
+    <joint name="wheel4_joint" type="continuous">
+        <parent link="body_link" />
+        <child link="wheel4_link" />
+        <origin
+            xyz="${body_link_x_dim/2 -1.2*wheel_link_radius} ${body_link_y_dim/2+wheel_link_length/2} ${wheel_link_z_location}"
+            rpy="0 0 0" />
+        <axis xyz="0 1 0" />
+        <limit effort="1000" velocity="1000" />
+        <dynamics damping="1.0" friction="1.0" />
+    </joint>
+    <link name="wheel4_link">
+        <visual>
+            <geometry>
+                <cylinder length="${wheel_link_length}" radius="${wheel_link_radius}" />
+            </geometry>
+            <origin rpy="${pi_const/2} 0 0" xyz="0 0 0" />
+        </visual>
+        <collision>
+            <geometry>
+                <cylinder length="${wheel_link_length}" radius="${wheel_link_radius}" />
+            </geometry>
+            <origin rpy="${pi_const/2} 0 0" xyz="0 0 0" />
+        </collision>
+        <xacro:inertia_wheel />
+    </link>
+    <!-- ####################### -->
+    <!-- END: Left front wheel and joint-->
+    <!-- ####################### -->
+    <joint name="wheel5_joint" type="continuous">
+        <parent link="body_link" />
+        <child link="wheel5_link" />
+        <origin
+            xyz="0 0 ${wheel_link_z_location}"
+            rpy="0 0 0" />
+        <axis xyz="0 1 0" />
+        <limit effort="1000" velocity="1000" />
+        <dynamics damping="1.0" friction="1.0" />
+    </joint>
+    <link name="wheel5_link">
+        <visual>
+            <geometry>
+                <cylinder length="${wheel_link_length}" radius="${wheel_link_radius}" />
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
File: src/mobile_robot/model/robot.xacro (robot description, xacro)
@@ -203,4 +203,29 @@
     <!-- END: Left front wheel and joint-->
     <!-- ####################### -->
+    <joint name="wheel5_joint" type="continuous">
+        <parent link="body_link" />
+        <child link="wheel5_link" />
+        <origin
+            xyz="0 0 ${wheel_link_z_location}"
+            rpy="0 0 0" />
+        <axis xyz="0 1 0" />
+        <limit effort="1000" velocity="1000" />
+        <dynamics damping="1.0" friction="1.0" />
+    </joint>
+    <link name="wheel5_link">
+        <visual>
+            <geometry>
+                <cylinder length="${wheel_link_length}" radius="${wheel_link_radius}" />
+            </geometry>
+            <origin rpy="${pi_const/2} 0 0" xyz="0 0 0" />
+        </visual>
+        <collision>
+            <geometry>
+                <cylinder length="${wheel_link_length}" radius="${wheel_link_radius}" />
+            </geometry>
+            <origin rpy="${pi_const/2} 0 0" xyz="0 0 0" />
+        </collision>
+        <xacro:inertia_wheel />
+    </link>
     <!-- ####################### -->
     <!-- Camera Link -->
