Commit message: now working 4 legs

File: install/mobile_robot/share/mobile_robot/model/robot.xacro (robot description, xacro)
@@ -5,4 +5,5 @@
 <!-- ####################### -->
 <robot name="differential_drive_robot" xmlns:xacro="http://www.ros.org/wiki/xacro">
+    <xacro:property name="scale" value=".005" />
     <!-- Body Dimensions -->
     <xacro:property name="body_link_x_dim" value="1" />
@@ -95,13 +96,15 @@
         <visual>
             <geometry>
-                <cylinder length="${wheel_link_length}" radius="${wheel_link_radius}" />
-            </geometry>
-            <origin rpy="${pi_const/2} 0 0" xyz="0 0 0" />
-        </visual>
-        <collision>
-            <geometry>
-                <cylinder length="${wheel_link_length}" radius="${wheel_link_radius}" />
-            </geometry>
-            <origin rpy="${pi_const/2} 0 0" xyz="0 0 0" />
+                <mesh filename="$(find mobile_robot)/meshes/lunar_zebro_legs.dae"
+                    scale="${scale} ${scale} ${scale}" />
+            </geometry>
+            <origin rpy="0 0 0" xyz="0 0 0" />
+        </visual>
+        <collision>
+            <geometry>
+                <mesh filename="$(find mobile_robot)/meshes/lunar_zebro_legs.dae"
+                    scale="${scale} ${scale} ${scale}" />
+            </geometry>
+            <origin rpy="0 0 0" xyz="0 0 0" />
         </collision>
         <xacro:inertia_wheel />
@@ -126,13 +129,15 @@
         <visual>
             <geometry>
-                <cylinder length="${wheel_link_length}" radius="${wheel_link_radius}" />
-            </geometry>
-            <origin rpy="${pi_const/2} 0 0" xyz="0 0 0" />
-        </visual>
-        <collision>
-            <geometry>
-                <cylinder length="${wheel_link_length}" radius="${wheel_link_radius}" />
-            </geometry>
-            <origin rpy="${pi_const/2} 0 0" xyz="0 0 0" />
+                <mesh filename="$(find mobile_robot)/meshes/lunar_zebro_legs.dae"
+                    scale="${scale} ${scale} ${scale}" />
+            </geometry>
+            <origin rpy="0 0 0" xyz="0 0 0" />
+        </visual>
+        <collision>
+            <geometry>
+                <mesh filename="$(find mobile_robot)/meshes/lunar_zebro_legs.dae"
+                    scale="${scale} ${scale} ${scale}" />
+            </geometry>
+            <origin rpy="0 0 0" xyz="0 0 0" />
         </collision>
         <xacro:inertia_wheel />
@@ -157,13 +162,15 @@
         <visual>
             <geometry>
-                <cylinder length="${wheel_link_length}" radius="${wheel_link_radius}" />
-            </geometry>
-            <origin rpy="${pi_const/2} 0 0" xyz="0 0 0" />
-        </visual>
-        <collision>
-            <geometry>
-                <cylinder length="${wheel_link_length}" radius="${wheel_link_radius}" />
-            </geometry>
-            <origin rpy="${pi_const/2} 0 0" xyz="0 0 0" />
+                <mesh filename="$(find mobile_robot)/meshes/lunar_zebro_legs.dae"
+                    scale="${scale} ${scale} ${scale}" />
+            </geometry>
+            <origin rpy="0 0 0" xyz="0 0 0" />
+        </visual>
+        <collision>
+            <geometry>
+                <mesh filename="$(find mobile_robot)/meshes/lunar_zebro_legs.dae"
+                    scale="${scale} ${scale} ${scale}" />
+            </geometry>
+            <origin rpy="0 0 0" xyz="0 0 0" />
         </collision>
         <xacro:inertia_wheel />
@@ -188,13 +195,15 @@
         <visual>
             <geometry>
-                <cylinder length="${wheel_link_length}" radius="${wheel_link_radius}" />
-            </geometry>
-            <origin rpy="${pi_const/2} 0 0" xyz="0 0 0" />
-        </visual>
-        <collision>
-            <geometry>
-                <cylinder length="${wheel_link_length}" radius="${wheel_link_radius}" />
-            </geometry>
-            <origin rpy="${pi_const/2} 0 0" xyz="0 0 0" />
+                <mesh filename="$(find mobile_robot)/meshes/lunar_zebro_legs.dae"
+                    scale="${scale} ${scale} ${scale}" />
+            </geometry>
+            <origin rpy="0 0 0" xyz="0 0 0" />
+        </visual>
+        <collision>
+            <geometry>
+                <mesh filename="$(find mobile_robot)/meshes/lunar_zebro_legs.dae"
+                    scale="${scale} ${scale} ${scale}" />
+            </geometry>
+            <origin rpy="0 0 0" xyz="0 0 0" />
         </collision>
         <xacro:inertia_wheel />
@@ -203,29 +212,4 @@
     <!-- END: Left front wheel and joint-->
     <!-- ####################### -->
-    <joint name="wheel5_joint" type="continuous">
-        <parent link="body_link" />
-        <child link="wheel5_link" />
-        <origin
-            xyz="0 0 ${wheel_link_z_location}"
-            rpy="0 0 0" />
-        <axis xyz="0 1 0" />
-        <limit effort="1000" velocity="1000" />
-        <dynamics damping="1.0" friction="1.0" />
-    </joint>
-    <link name="wheel5_link">
-        <visual>
-            <geometry>
-                <cylinder length="${wheel_link_length}" radius="${wheel_link_radius}" />
-            </geometry>
-            <origin rpy="${pi_const/2} 0 0" xyz="0 0 0" />
-        </visual>
-        <collision>
-            <geometry>
-                <cylinder length="${wheel_link_length}" radius="${wheel_link_radius}" />
-            </geometry>
-            <origin rpy="${pi_const/2} 0 0" xyz="0 0 0" />
-        </collision>
-        <xacro:inertia_wheel />
-    </link>
     <!-- ####################### -->
     <!-- Camera Link -->
@@ -248,5 +232,4 @@
                 <box size="${camera_link} ${camera_link} ${camera_link}" />
             </geometry>
-            <material name="red" />
         </visual>
         <inertial>

Commit message: now working 6 legs

File: install/mobile_robot/share/mobile_robot/model/robot.xacro (robot description, xacro)
@@ -29,4 +29,6 @@
         value="${(1.0/12.0)*wheel_mass*(3.0*wheel_link_radius*wheel_link_radius+wheel_link_length*wheel_link_length)}" />
     <xacro:property name="camera_link" value="0.05" /> <!-- Size of square 'camera' box -->
+<!--    middle wheel offset-->
+        <xacro:property name="middle_wheel_extra_offset" value="0.1" />
     <!-- This macro defines the inertial section of the wheel -->
     <xacro:macro name="inertia_wheel">
@@ -99,12 +101,12 @@
                     scale="${scale} ${scale} ${scale}" />
             </geometry>
-            <origin rpy="0 0 0" xyz="0 0 0" />
-        </visual>
-        <collision>
-            <geometry>
-                <mesh filename="$(find mobile_robot)/meshes/lunar_zebro_legs.dae"
-                    scale="${scale} ${scale} ${scale}" />
-            </geometry>
-            <origin rpy="0 0 0" xyz="0 0 0" />
+            <origin rpy="0 0 ${pi_const}" xyz="0 0 0" />
+        </visual>
+        <collision>
+            <geometry>
+                <mesh filename="$(find mobile_robot)/meshes/lunar_zebro_legs.dae"
+                    scale="${scale} ${scale} ${scale}" />
+            </geometry>
+            <origin rpy="0 0 ${pi_const}" xyz="0 0 0" />
         </collision>
         <xacro:inertia_wheel />
@@ -132,12 +134,12 @@
                     scale="${scale} ${scale} ${scale}" />
             </geometry>
-            <origin rpy="0 0 0" xyz="0 0 0" />
-        </visual>
-        <collision>
-            <geometry>
-                <mesh filename="$(find mobile_robot)/meshes/lunar_zebro_legs.dae"
-                    scale="${scale} ${scale} ${scale}" />
-            </geometry>
-            <origin rpy="0 0 0" xyz="0 0 0" />
+            <origin rpy="0 0 ${pi_const}" xyz="0 0 0" />
+        </visual>
+        <collision>
+            <geometry>
+                <mesh filename="$(find mobile_robot)/meshes/lunar_zebro_legs.dae"
+                    scale="${scale} ${scale} ${scale}" />
+            </geometry>
+            <origin rpy="0 0 ${pi_const}" xyz="0 0 0" />
         </collision>
         <xacro:inertia_wheel />
@@ -165,12 +167,12 @@
                     scale="${scale} ${scale} ${scale}" />
             </geometry>
-            <origin rpy="0 0 0" xyz="0 0 0" />
-        </visual>
-        <collision>
-            <geometry>
-                <mesh filename="$(find mobile_robot)/meshes/lunar_zebro_legs.dae"
-                    scale="${scale} ${scale} ${scale}" />
-            </geometry>
-            <origin rpy="0 0 0" xyz="0 0 0" />
+            <origin rpy="0 0 ${pi_const}" xyz="0 0 0" />
+        </visual>
+        <collision>
+            <geometry>
+                <mesh filename="$(find mobile_robot)/meshes/lunar_zebro_legs.dae"
+                    scale="${scale} ${scale} ${scale}" />
+            </geometry>
+            <origin rpy="0 0 ${pi_const}" xyz="0 0 0" />
         </collision>
         <xacro:inertia_wheel />
@@ -198,12 +200,61 @@
                     scale="${scale} ${scale} ${scale}" />
             </geometry>
-            <origin rpy="0 0 0" xyz="0 0 0" />
-        </visual>
-        <collision>
-            <geometry>
-                <mesh filename="$(find mobile_robot)/meshes/lunar_zebro_legs.dae"
-                    scale="${scale} ${scale} ${scale}" />
-            </geometry>
-            <origin rpy="0 0 0" xyz="0 0 0" />
+            <origin rpy="0 0 ${pi_const}" xyz="0 0 0" />
+        </visual>
+        <collision>
+            <geometry>
+                <mesh filename="$(find mobile_robot)/meshes/lunar_zebro_legs.dae"
+                    scale="${scale} ${scale} ${scale}" />
+            </geometry>
+            <origin rpy="0 0 ${pi_const}" xyz="0 0 0" />
+        </collision>
+        <xacro:inertia_wheel />
+    </link>
+    <joint name="wheel5_joint" type="continuous">
+        <parent link="body_link" />
+        <child link="wheel5_link" />
+        <origin xyz="0 ${-body_link_y_dim/2-wheel_link_length/2-middle_wheel_extra_offset} ${wheel_link_z_location}" rpy="0 0 0" />
+        <axis xyz="0 1 0" />
+        <limit effort="1000" velocity="1000" />
+        <dynamics damping="1.0" friction="1.0" />
+    </joint>
+    <link name="wheel5_link">
+        <visual>
+            <geometry>
+                <mesh filename="$(find mobile_robot)/meshes/lunar_zebro_legs.dae" scale="${scale} ${scale} ${scale}" />
+            </geometry>
+            <origin rpy="0 0 ${pi_const}" xyz="0 0 0" />
+        </visual>
+        <collision>
+            <geometry>
+                <mesh filename="$(find mobile_robot)/meshes/lunar_zebro_legs.dae" scale="${scale} ${scale} ${scale}" />
+            </geometry>
+            <origin rpy="0 0 ${pi_const}" xyz="0 0 0" />
+        </collision>
+        <xacro:inertia_wheel />
+    </link>
+    <!-- ####################### -->
+    <!-- Start: Middle left wheel of the robot and the joint-->
+    <!-- ####################### -->
+    <joint name="wheel6_joint" type="continuous">
+        <parent link="body_link" />
+        <child link="wheel6_link" />
+        <origin xyz="0 ${body_link_y_dim/2+wheel_link_length/2+middle_wheel_extra_offset} ${wheel_link_z_location}" rpy="0 0 0" />
+        <axis xyz="0 1 0" />
+        <limit effort="1000" velocity="1000" />
+        <dynamics damping="1.0" friction="1.0" />
+    </joint>
+    <link name="wheel6_link">
+        <visual>
+            <geometry>
+                <mesh filename="$(find mobile_robot)/meshes/lunar_zebro_legs.dae" scale="${scale} ${scale} ${scale}" />
+            </geometry>
+            <origin rpy="0 0 ${pi_const}" xyz="0 0 0" />
+        </visual>
+        <collision>
+            <geometry>
+                <mesh filename="$(find mobile_robot)/meshes/lunar_zebro_legs.dae" scale="${scale} ${scale} ${scale}" />
+            </geometry>
+            <origin rpy="0 0 ${pi_const}" xyz="0 0 0" />
         </collision>
         <xacro:inertia_wheel />
